File: pwm_module_sch/pwm_module_sch.sch (KiCad schematic (older format))
At the start: 55 parts, among them J1 SWIMM, J2 output -, J3 input, J4 output+, J5 uart, Q1 AO3400, Q2 IRFZ44N, SW1 ., SW2 ., U1 TM1637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

Commit message: board fixed
Parts:
- removed D5, D6, D7, D9: ., Package_TO_SOT_THT:TO-220-3_Vertical, symbol pwm_module_sch-rescue:D_Schottky_Dual_CommonCathode_AKA-Device-pwm_module_sch-r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
- removed RV1, RV2: ., pwm_module:SP3-4, symbol pwm_module_sch-rescue:R_Potentiometer-Device-pwm_module_sch-rescue
- added D5, D6, D7, D9: ., Package_TO_SOT_THT:TO-220-3_Vertical, symbol Device:D_Schottky_Dual_CommonCathode_AKA_Parallel
- added RV1, RV2: ., pwm_module:SP3-4, symbol Device:R_Potentiometer
- C5, C6: symbol pwm_module_sch-rescue:C_Polarized_US-Device-pwm_module_sch-rescue -> Device:C_Polarized
Connections:
- net +24V: now also D9.2 (A)
- net +3V3: now also RV1.3, RV2.3
- net GND: now also D5.1 (K), D5.3 (K), D6.1 (K), D6.3 (K), D7.1 (K), D7.3 (K), RV1.1, RV2.1
- net at J3.1 (Pin_1): now also D6.2 (A), D9.1 (K)
- net at J3.2 (Pin_2): now also D7.2 (A), D9.3 (K)
- net at L1.1, Q2.3 (S): now also D5.2 (A)
- net at C14.1, R15.2: now also RV1.2
- net at C13.1, R16.1: now also RV2.2
Other:
- moved on the sheet: C7, C8, C9, D8, R8, U4
